Commit message: Changing licenses in the big '26

File: dx_description/dx_e3r3_finger.urdf (robot description, URDF)
Before this commit: robot dx_e3r3_finger, 5 links, 4 joints
Links:
- link F0_J0_link: geometry collision mesh filename=package://dx_description/meshes/dx_e3r3_finger/F0_J0_link.S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; visual mesh filename=package://dx_description/meshes/dx_e3r3_finger/F0_J0_link.S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
- link F0_base: geometry collision mesh filename=package://dx_description/meshes/dx_e3r3_finger/F0_base.STL; visual mesh filename=package://dx_description/meshes/dx_e3r3_finger/F0_base.STL
- link F0_distal: geometry collision mesh filename=package://dx_description/meshes/dx_e3r3_finger/F0_distal.STL; visual mesh filename=package://dx_description/meshes/dx_e3r3_finger/F0_distal.STL
- link F0_middle: geometry collision mesh filename=package://dx_description/meshes/dx_e3r3_finger/F0_middle.STL; visual mesh filename=package://dx_description/meshes/dx_e3r3_finger/F0_middle.STL
- link F0_proximal: geometry collision mesh filename=package://dx_description/meshes/dx_e3r3_finger/F0_proximal.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; visual mesh filename=package://dx_description/meshes/dx_e3r3_finger/F0_proximal.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

File: dx_description/robot/0x02000105.urdf.xacro (robot description, xacro)
@@ -1,6 +1,26 @@
 <?xml version="1.0" encoding="utf-8"?>
 <!--
- Copyright (C) 2024-2026 Shadow Robot Company Ltd - All Rights Reserved. Proprietary and Confidential.
- Unauthorized copying of the content in this file, via any medium is strictly prohibited.
+ Software License Agreement (BSD License)
+ Copyright © 2026 belongs to Shadow Robot Company Ltd.
+ All rights reserved.
+ Redistribution and use in source and binary forms, with or without modification,
+ are permitted provided that the following conditions are met:
+   1. Redistributions of source code must retain the above copyright notice,
+      this list of conditions and the following disclaimer.
+   2. Redistributions in binary form must reproduce the above copyright notice,
+      this list of conditions and the following disclaimer in the documentation
+      and/or other materials provided with the distribution.
+   3. Neither the name of Shadow Robot Company Ltd nor the names of its contributors
+      may be used to endorse or promote products derived from this software without
+      specific prior written permission.
+ This software is provided by Shadow Robot Company Ltd "as is" and any express
+ or implied warranties, including, but not limited to, the implied warranties of
+ merchantability and fitness for a particular purpose are disclaimed. In no event
+ shall the copyright holder be liable for any direct, indirect, incidental, special,
+ exemplary, or consequential damages (including, but not limited to, procurement of
+ substitute goods or services; loss of use, data, or profits; or business interruption)
+ however caused and on any theory of liability, whether in contract, strict liability,
+ or tort (including negligence or otherwise) arising in any way out of the use of this
+ software, even if advised of the possibility of such damage.
 -->
 <robot name="e3_r3_hand" xmlns:xacro="http://www.ros.org/wiki/xacro">

File: dx_description/robot/0x02000105.xacro (robot description, xacro)
@@ -1,6 +1,26 @@
 <?xml version="1.0" encoding="utf-8"?>
 <!--
- Copyright (C) 2024-2026 Shadow Robot Company Ltd - All Rights Reserved. Proprietary and Confidential.
- Unauthorized copying of the content in this file, via any medium is strictly prohibited.
+ Software License Agreement (BSD License)
+ Copyright © 2026 belongs to Shadow Robot Company Ltd.
+ All rights reserved.
+ Redistribution and use in source and binary forms, with or without modification,
+ are permitted provided that the following conditions are met:
+   1. Redistributions of source code must retain the above copyright notice,
+      this list of conditions and the following disclaimer.
+   2. Redistributions in binary form must reproduce the above copyright notice,
+      this list of conditions and the following disclaimer in the documentation
+      and/or other materials provided with the distribution.
+   3. Neither the name of Shadow Robot Company Ltd nor the names of its contributors
+      may be used to endorse or promote products derived from this software without
+      specific prior written permission.
+ This software is provided by Shadow Robot Company Ltd "as is" and any express
+ or implied warranties, including, but not limited to, the implied warranties of
+ merchantability and fitness for a particular purpose are disclaimed. In no event
+ shall the copyright holder be liable for any direct, indirect, incidental, special,
+ exemplary, or consequential damages (including, but not limited to, procurement of
+ substitute goods or services; loss of use, data, or profits; or business interruption)
+ however caused and on any theory of liability, whether in contract, strict liability,
+ or tort (including negligence or otherwise) arising in any way out of the use of this
+ software, even if advised of the possibility of such damage.
 -->
 <robot name="e3_r3_hand" xmlns:xacro="http://ros.org/wiki/xacro">

File: dx_description/robot/0x02000106.urdf.xacro (robot description, xacro)
@@ -1,6 +1,26 @@
 <?xml version="1.0" encoding="utf-8"?>
 <!--
- Copyright (C) 2025-2026 Shadow Robot Company Ltd - All Rights Reserved. Proprietary and Confidential.
- Unauthorized copying of the content in this file, via any medium is strictly prohibited.
+ Software License Agreement (BSD License)
+ Copyright © 2026 belongs to Shadow Robot Company Ltd.
+ All rights reserved.
+ Redistribution and use in source and binary forms, with or without modification,
+ are permitted provided that the following conditions are met:
+   1. Redistributions of source code must retain the above copyright notice,
+      this list of conditions and the following disclaimer.
+   2. Redistributions in binary form must reproduce the above copyright notice,
+      this list of conditions and the following disclaimer in the documentation
+      and/or other materials provided with the distribution.
+   3. Neither the name of Shadow Robot Company Ltd nor the names of its contributors
+      may be used to endorse or promote products derived from this software without
+      specific prior written permission.
+ This software is provided by Shadow Robot Company Ltd "as is" and any express
+ or implied warranties, including, but not limited to, the implied warranties of
+ merchantability and fitness for a particular purpose are disclaimed. In no event
+ shall the copyright holder be liable for any direct, indirect, incidental, special,
+ exemplary, or consequential damages (including, but not limited to, procurement of
+ substitute goods or services; loss of use, data, or profits; or business interruption)
+ however caused and on any theory of liability, whether in contract, strict liability,
+ or tort (including negligence or otherwise) arising in any way out of the use of this
+ software, even if advised of the possibility of such damage.
 -->
 <robot name="e3_r3_hand" xmlns:xacro="http://www.ros.org/wiki/xacro">

File: dx_description/robot/0x02000106.xacro (robot description, xacro)
@@ -1,6 +1,26 @@
 <?xml version="1.0" encoding="utf-8"?>
 <!--
- Copyright (C) 2024-2026 Shadow Robot Company Ltd - All Rights Reserved. Proprietary and Confidential.
- Unauthorized copying of the content in this file, via any medium is strictly prohibited.
+ Software License Agreement (BSD License)
+ Copyright © 2026 belongs to Shadow Robot Company Ltd.
+ All rights reserved.
+ Redistribution and use in source and binary forms, with or without modification,
+ are permitted provided that the following conditions are met:
+   1. Redistributions of source code must retain the above copyright notice,
+      this list of conditions and the following disclaimer.
+   2. Redistributions in binary form must reproduce the above copyright notice,
+      this list of conditions and the following disclaimer in the documentation
+      and/or other materials provided with the distribution.
+   3. Neither the name of Shadow Robot Company Ltd nor the names of its contributors
+      may be used to endorse or promote products derived from this software without
+      specific prior written permission.
+ This software is provided by Shadow Robot Company Ltd "as is" and any express
+ or implied warranties, including, but not limited to, the implied warranties of
+ merchantability and fitness for a particular purpose are disclaimed. In no event
+ shall the copyright holder be liable for any direct, indirect, incidental, special,
+ exemplary, or consequential damages (including, but not limited to, procurement of
+ substitute goods or services; loss of use, data, or profits; or business interruption)
+ however caused and on any theory of liability, whether in contract, strict liability,
+ or tort (including negligence or otherwise) arising in any way out of the use of this
+ software, even if advised of the possibility of such damage.
 -->
 <robot name="e3_r3_hand" xmlns:xacro="http://ros.org/wiki/xacro">

File: dx_description/xacros/dx_e3r3_finger.xacro (robot description, xacro)
@@ -1,6 +1,26 @@
 <?xml version="1.0" encoding="utf-8"?>
 <!--
- Copyright (C) 2024-2026 Shadow Robot Company Ltd - All Rights Reserved. Proprietary and Confidential.
- Unauthorized copying of the content in this file, via any medium is strictly prohibited.
+ Software License Agreement (BSD License)
+ Copyright © 2026 belongs to Shadow Robot Company Ltd.
+ All rights reserved.
+ Redistribution and use in source and binary forms, with or without modification,
+ are permitted provided that the following conditions are met:
+   1. Redistributions of source code must retain the above copyright notice,
+      this list of conditions and the following disclaimer.
+   2. Redistributions in binary form must reproduce the above copyright notice,
+      this list of conditions and the following disclaimer in the documentation
+      and/or other materials provided with the distribution.
+   3. Neither the name of Shadow Robot Company Ltd nor the names of its contributors
+      may be used to endorse or promote products derived from this software without
+      specific prior written permission.
+ This software is provided by Shadow Robot Company Ltd "as is" and any express
+ or implied warranties, including, but not limited to, the implied warranties of
+ merchantability and fitness for a particular purpose are disclaimed. In no event
+ shall the copyright holder be liable for any direct, indirect, incidental, special,
+ exemplary, or consequential damages (including, but not limited to, procurement of
+ substitute goods or services; loss of use, data, or profits; or business interruption)
+ however caused and on any theory of liability, whether in contract, strict liability,
+ or tort (including negligence or otherwise) arising in any way out of the use of this
+ software, even if advised of the possibility of such damage.
 -->
 <robot xmlns:xacro="http://ros.org/wiki/xacro">

File: dx_description/xacros/mounting_plates/G-SHW063_Tool_change_plate.xacro (robot description, xacro)
@@ -1,6 +1,26 @@
 <?xml version="1.0" encoding="utf-8"?>
 <!--
- Copyright (C) 2025-2026 Shadow Robot Company Ltd - All Rights Reserved. Proprietary and Confidential.
- Unauthorized copying of the content in this file, via any medium is strictly prohibited.
+ Software License Agreement (BSD License)
+ Copyright © 2026 belongs to Shadow Robot Company Ltd.
+ All rights reserved.
+ Redistribution and use in source and binary forms, with or without modification,
+ are permitted provided that the following conditions are met:
+   1. Redistributions of source code must retain the above copyright notice,
+      this list of conditions and the following disclaimer.
+   2. Redistributions in binary form must reproduce the above copyright notice,
+      this list of conditions and the following disclaimer in the documentation
+      and/or other materials provided with the distribution.
+   3. Neither the name of Shadow Robot Company Ltd nor the names of its contributors
+      may be used to endorse or promote products derived from this software without
+      specific prior written permission.
+ This software is provided by Shadow Robot Company Ltd "as is" and any express
+ or implied warranties, including, but not limited to, the implied warranties of
+ merchantability and fitness for a particular purpose are disclaimed. In no event
+ shall the copyright holder be liable for any direct, indirect, incidental, special,
+ exemplary, or consequential damages (including, but not limited to, procurement of
+ substitute goods or services; loss of use, data, or profits; or business interruption)
+ however caused and on any theory of liability, whether in contract, strict liability,
+ or tort (including negligence or otherwise) arising in any way out of the use of this
+ software, even if advised of the possibility of such damage.
 -->
 <robot xmlns:xacro="http://ros.org/wiki/xacro">
