Commit message: Added distac xacro, meshes

File: dx_description/robot/0x02000105.urdf.xacro (robot description, xacro)
@@ -27,4 +27,5 @@
   <xacro:include filename="$(find dx_description)/robot/0x02000105.xacro" />
   <xacro:arg name="prefix" default="" />
+  <xacro:arg name="distal_type" default="sparkle" />  <!-- "sparkle" or "magtac" -->
   <link name="world" />
   <joint name="$(arg prefix)world_joint" type="fixed">

File: dx_description/robot/0x02000105.xacro (robot description, xacro)
@@ -25,5 +25,5 @@
 -->
 <robot name="dexee_config_1_hand" xmlns:xacro="http://ros.org/wiki/xacro">
-  <xacro:macro name="dexee_config_1_hand" params="prefix:=^">
+  <xacro:macro name="dexee_config_1_hand" params="prefix:=^ distal_type:=^">
     <link name="${prefix}hand_base">
       <inertial>

File: dx_description/robot/0x02000106.urdf.xacro (robot description, xacro)
@@ -27,6 +27,7 @@
   <xacro:include filename="$(find dx_description)/robot/0x02000106.xacro" />
   <xacro:arg name="prefix" default="" />
+  <xacro:arg name="distal_type" default="sparkle" />  <!-- "sparkle" or "magtac" -->
   <link name="world" />
-  <xacro:dexee_config_1_hand prefix="$(arg prefix)" />
+  <xacro:dexee_config_1_hand prefix="$(arg prefix)" distal_type="$(arg distal_type)" />
   <gazebo>
     <plugin name="gazebo_ros_control" filename="libgazebo_ros_control.so">

File: dx_description/robot/0x02000106.xacro (robot description, xacro)
@@ -25,5 +25,5 @@
 -->
 <robot name="dexee_config_1_hand" xmlns:xacro="http://ros.org/wiki/xacro">
-  <xacro:macro name="dexee_config_1_hand" params="prefix:=^">
+  <xacro:macro name="dexee_config_1_hand" params="prefix:=^ distal_type:=^">
     <xacro:include filename="$(find dx_description)/xacros/dx_e3r3_finger.xacro" />
     <xacro:macro_e3r3_finger prefix="${prefix}" finger_id="F0" parent="world">

File: dx_description/robot/0x02000107.urdf.xacro (robot description, xacro)
@@ -27,4 +27,5 @@
   <xacro:include filename="$(find dx_description)/robot/0x02000107.xacro" />
   <xacro:arg name="prefix" default="" />
+  <xacro:arg name="distal_type" default="sparkle" />  <!-- "sparkle" or "magtac" -->
   <link name="world" />
   <joint name="$(arg prefix)world_joint" type="fixed">
@@ -32,5 +33,5 @@
     <child link="$(arg prefix)hand_base" />
   </joint>
-  <xacro:dexee_config_2_right_hand prefix="$(arg prefix)" />
+  <xacro:dexee_config_2_right_hand prefix="$(arg prefix)"/>
   <gazebo>
     <plugin name="gazebo_ros_control" filename="libgazebo_ros_control.so">

File: dx_description/robot/0x02000107.xacro (robot description, xacro)
@@ -25,5 +25,5 @@
 -->
 <robot name="dexee_config_2_right_hand" xmlns:xacro="http://ros.org/wiki/xacro">
-  <xacro:macro name="dexee_config_2_right_hand" params="prefix:=^">
+  <xacro:macro name="dexee_config_2_right_hand" params="prefix:=^ distal_type:=^">
     <link name="${prefix}hand_base">
       <inertial>

File: dx_description/robot/0x02000109.urdf.xacro (robot description, xacro)
@@ -27,4 +27,5 @@
   <xacro:include filename="$(find dx_description)/robot/0x02000109.xacro" />
   <xacro:arg name="prefix" default="" />
+  <xacro:arg name="distal_type" default="sparkle" />  <!-- "sparkle" or "magtac" -->
   <link name="world" />
   <joint name="$(arg prefix)world_joint" type="fixed">

File: dx_description/xacros/distals/magtac.xacro (robot description, xacro)
@@ -24,20 +24,19 @@
  software, even if advised of the possibility of such damage.
 -->
-<robot name="dexee_config_2_left_hand" xmlns:xacro="http://ros.org/wiki/xacro">
-  <xacro:macro name="dexee_config_2_left_hand" params="prefix:=^ distal_type:=^">
-    <link name="${prefix}hand_base">
+<robot xmlns:xacro="http://ros.org/wiki/xacro">
+  <xacro:macro name="macro_e3r3_distal" params="prefix:=^ finger_id:=^ parent">
+    <link name="${prefix}${finger_id}_distal">
       <inertial>
-        <origin xyz="0.0176605661792342 -0.040301709672928 0.0592639986942411" rpy="0 0 0" />
-        <mass value="0.53506724" />
-        <inertia ixx="0.00362636445124211" ixy="0.000732417243232051" ixz="-0.000377582935294335"
-                 iyy="0.00200238966610271" iyz="-3.61002555746394E-05" izz="0.00423035114084856" />
+        <origin xyz="0.00084325 0.00164346 0.01482169" rpy="0 0 0" />
+        <mass value="0.02766365" />
+        <inertia ixx="0.0000051" ixy="0" ixz="0.00000028" iyy="0.00000506" iyz="-0.00000034" izz="0.00000198" />
       </inertial>
       <visual>
         <origin xyz="0 0 0" rpy="0 0 0" />
         <geometry>
-          <mesh filename="package://dx_description/meshes/hand_bases/Config_2_Left_Hand_Base.dae" />
+            <mesh filename="package://dx_description/meshes/distal/magtac.dae" />
         </geometry>
         <material name="">
-          <color rgba="0.898039215686275 0.917647058823529 0.929411764705882 1" />
+          <color rgba="0.75294 0.75294 0.75294 1" />
         </material>
       </visual>
@@ -45,28 +44,25 @@
         <origin xyz="0 0 0" rpy="0 0 0" />
         <geometry>
-          <mesh filename="package://dx_description/meshes/hand_bases/collision/Config_2_Left_Hand_Base.stl" />
+          <mesh filename="package://dx_description/meshes/distals/collision/magtac.stl" />
         </geometry>
       </collision>
     </link>
-    <gazebo reference="${prefix}hand_base">
+    <gazebo reference="${prefix}${finger_id}_distal">
       <selfCollide>true</selfCollide>
     </gazebo>
-    <!-- Create a virtual end effector link that will be useful for arm IK -->
-    <link name="${prefix}end_effector"/>
-    <joint name="${prefix}ee_fixed_joint" type="fixed">
-      <parent link="${prefix}hand_base"/>
-      <child link="${prefix}end_effector"/>
-      <origin rpy="0.0 0.0 0.0" xyz="0.0 0.0 0.25"/>
+    <joint name="${prefix}${finger_id}_J3" type="revolute">
+      <origin xyz="0 0 0.035" rpy="0 0 0" />
+      <parent link="${parent}" />
+      <child link="${prefix}${finger_id}_distal" />
+      <axis xyz="1 0 0" />
+      <limit lower="-0.523" upper="1.485" effort="0.35" velocity="3.1415" />
+      <dynamics friction="0.001"/>
     </joint>
-    <xacro:include filename="$(find dx_description)/xacros/dx_e3r3_finger.xacro" />
-    <xacro:macro_e3r3_finger prefix="${prefix}" finger_id="F0" parent="${prefix}hand_base">
-      <origin xyz="0.0882673027707308 -0.12823624685039 0.0575255687317372" rpy="-1.74273004 -0.77031903 -1.32641633"/>
-    </xacro:macro_e3r3_finger>
-    <xacro:macro_e3r3_finger prefix="${prefix}" finger_id="F1" parent="${prefix}hand_base">
-      <origin xyz="0.0495780670511493 -0.0794348993309075 0.00872422121225381" rpy="-2.22448705 -0.47183267 -0.5355029"/>
-    </xacro:macro_e3r3_finger>
-    <xacro:macro_e3r3_finger prefix="${prefix}" finger_id="F2" parent="${prefix}hand_base">
-      <origin xyz="-0.0375495099984522 -0.105081515549682 0.00891499330831318" rpy="-1.57079633  0.78539816  1.57079633"/>
-    </xacro:macro_e3r3_finger>
+    <link name="${prefix}${finger_id}_tip" />
+    <joint name="${prefix}${finger_id}_distal_tip" type="fixed">
+        <parent link="${prefix}${finger_id}_distal" />
+        <child link="${prefix}${finger_id}_tip" />
+        <origin xyz="0 0.003 0.033" rpy="0 0 0" />
+    </joint>
   </xacro:macro>
 </robot>

File: dx_description/xacros/distals/sparkle.xacro (robot description, xacro)
@@ -24,20 +24,19 @@
  software, even if advised of the possibility of such damage.
 -->
-<robot name="dexee_config_2_left_hand" xmlns:xacro="http://ros.org/wiki/xacro">
-  <xacro:macro name="dexee_config_2_left_hand" params="prefix:=^ distal_type:=^">
-    <link name="${prefix}hand_base">
+<robot xmlns:xacro="http://ros.org/wiki/xacro">
+  <xacro:macro name="macro_e3r3_distal" params="prefix:=^ finger_id:=^ parent">
+    <link name="${prefix}${finger_id}_distal">
       <inertial>
-        <origin xyz="0.0176605661792342 -0.040301709672928 0.0592639986942411" rpy="0 0 0" />
-        <mass value="0.53506724" />
-        <inertia ixx="0.00362636445124211" ixy="0.000732417243232051" ixz="-0.000377582935294335"
-                 iyy="0.00200238966610271" iyz="-3.61002555746394E-05" izz="0.00423035114084856" />
+        <origin xyz="0.00084325 0.00164346 0.01482169" rpy="0 0 0" />
+        <mass value="0.02766365" />
+        <inertia ixx="0.0000051" ixy="0" ixz="0.00000028" iyy="0.00000506" iyz="-0.00000034" izz="0.00000198" />
       </inertial>
       <visual>
         <origin xyz="0 0 0" rpy="0 0 0" />
         <geometry>
-          <mesh filename="package://dx_description/meshes/hand_bases/Config_2_Left_Hand_Base.dae" />
+            <mesh filename="package://dx_description/meshes/distals/sparkle.dae" />
         </geometry>
         <material name="">
-          <color rgba="0.898039215686275 0.917647058823529 0.929411764705882 1" />
+          <color rgba="0.75294 0.75294 0.75294 1" />
         </material>
       </visual>
@@ -45,28 +44,25 @@
         <origin xyz="0 0 0" rpy="0 0 0" />
         <geometry>
-          <mesh filename="package://dx_description/meshes/hand_bases/collision/Config_2_Left_Hand_Base.stl" />
+          <mesh filename="package://dx_description/meshes/distals/collision/sparkle.stl" />
         </geometry>
       </collision>
     </link>
-    <gazebo reference="${prefix}hand_base">
+    <gazebo reference="${prefix}${finger_id}_distal">
       <selfCollide>true</selfCollide>
     </gazebo>
-    <!-- Create a virtual end effector link that will be useful for arm IK -->
-    <link name="${prefix}end_effector"/>
-    <joint name="${prefix}ee_fixed_joint" type="fixed">
-      <parent link="${prefix}hand_base"/>
-      <child link="${prefix}end_effector"/>
-      <origin rpy="0.0 0.0 0.0" xyz="0.0 0.0 0.25"/>
+    <joint name="${prefix}${finger_id}_J3" type="revolute">
+      <origin xyz="0 0 0.035" rpy="0 0 0" />
+      <parent link="${parent}" />
+      <child link="${prefix}${finger_id}_distal" />
+      <axis xyz="1 0 0" />
+      <limit lower="-0.523" upper="1.485" effort="0.35" velocity="3.1415" />
+      <dynamics friction="0.001"/>
     </joint>
-    <xacro:include filename="$(find dx_description)/xacros/dx_e3r3_finger.xacro" />
-    <xacro:macro_e3r3_finger prefix="${prefix}" finger_id="F0" parent="${prefix}hand_base">
-      <origin xyz="0.0882673027707308 -0.12823624685039 0.0575255687317372" rpy="-1.74273004 -0.77031903 -1.32641633"/>
-    </xacro:macro_e3r3_finger>
-    <xacro:macro_e3r3_finger prefix="${prefix}" finger_id="F1" parent="${prefix}hand_base">
-      <origin xyz="0.0495780670511493 -0.0794348993309075 0.00872422121225381" rpy="-2.22448705 -0.47183267 -0.5355029"/>
-    </xacro:macro_e3r3_finger>
-    <xacro:macro_e3r3_finger prefix="${prefix}" finger_id="F2" parent="${prefix}hand_base">
-      <origin xyz="-0.0375495099984522 -0.105081515549682 0.00891499330831318" rpy="-1.57079633  0.78539816  1.57079633"/>
-    </xacro:macro_e3r3_finger>
+    <link name="${prefix}${finger_id}_tip" />
+    <joint name="${prefix}${finger_id}_distal_tip" type="fixed">
+        <parent link="${prefix}${finger_id}_distal" />
+        <child link="${prefix}${finger_id}_tip" />
+        <origin xyz="0 0.003 0.033" rpy="0 0 0" />
+    </joint>
   </xacro:macro>
 </robot>

File: dx_description/xacros/dx_e3r3_finger.xacro (robot description, xacro)
@@ -25,5 +25,5 @@
 -->
 <robot xmlns:xacro="http://ros.org/wiki/xacro">
-  <xacro:macro name="macro_e3r3_finger" params="prefix:=^ finger_id parent *origin">
+  <xacro:macro name="macro_e3r3_finger" params="prefix:=^ distal_type:=^ finger_id parent *origin">
     <joint name="${prefix}world_joint_${finger_id}" type="fixed">
       <xacro:insert_block name="origin"/>
@@ -157,43 +157,6 @@
       <dynamics friction="0.001"/>
     </joint>
-    <link name="${prefix}${finger_id}_distal">
-      <inertial>
-        <origin xyz="0.00084325 0.00164346 0.01482169" rpy="0 0 0" />
-        <mass value="0.02766365" />
-        <inertia ixx="0.0000051" ixy="0" ixz="0.00000028" iyy="0.00000506" iyz="-0.00000034" izz="0.00000198" />
-      </inertial>
-      <visual>
-        <origin xyz="0 0 0" rpy="0 0 0" />
-        <geometry>
-            <mesh filename="package://dx_description/meshes/dx_e3r3_finger/F0_distal.dae" />
-        </geometry>
-        <material name="">
-          <color rgba="0.75294 0.75294 0.75294 1" />
-        </material>
-      </visual>
-      <collision>
-        <origin xyz="0 0 0" rpy="0 0 0" />
-        <geometry>
-          <mesh filename="package://dx_description/meshes/dx_e3r3_finger/collision/F0_distal.stl" />
-        </geometry>
-      </collision>
-    </link>
-    <gazebo reference="${prefix}${finger_id}_distal">
-      <selfCollide>true</selfCollide>
-    </gazebo>
-    <joint name="${prefix}${finger_id}_J3" type="revolute">
-      <origin xyz="0 0 0.035" rpy="0 0 0" />
-      <parent link="${prefix}${finger_id}_middle" />
-      <child link="${prefix}${finger_id}_distal" />
-      <axis xyz="1 0 0" />
-      <limit lower="-0.523" upper="1.485" effort="0.35" velocity="3.1415" />
-      <dynamics friction="0.001"/>
-    </joint>
-    <link name="${prefix}${finger_id}_tip" />
-    <joint name="${prefix}${finger_id}_distal_tip" type="fixed">
-        <parent link="${prefix}${finger_id}_distal" />
-        <child link="${prefix}${finger_id}_tip" />
-        <origin xyz="0 0.003 0.033" rpy="0 0 0" />
-    </joint>
+    <xacro:include filename="$(find dx_description)/xacros/distals/${distal_type}.xacro" />
+    <xacro:macro_e3r3_distal parent="${prefix}${finger_id}_middle"/>
     <!-- These transmissions are wrongly configured and fail to be loaded by the real robot -->
     <!-- We still need to define them in order to be able to launch the robot in simulation -->
