Commit message: Single finger URDF has a base and finger blanks

File: dx_description/robot/0x02000106.xacro (robot description, xacro)
@@ -26,8 +26,48 @@
 <robot name="dexee_config_1_hand" xmlns:xacro="http://ros.org/wiki/xacro">
   <xacro:macro name="dexee_config_1_hand" params="prefix:=^ distal_type:=^">
+    <link name="${prefix}hand_base">
+      <inertial>
+        <origin xyz="0.00024269 0.0064896 0.05011689" rpy="0 0 0" />
+        <mass value="0.53506724" />
+        <inertia ixx="0.00235606" ixy="-0.00000318" ixz="0.00001251"
+                 iyy="0.00262644" iyz="-0.00010584" izz="0.00095084" />
+      </inertial>
+      <visual>
+        <origin xyz="0 0 0" rpy="0 0 0" />
+        <geometry>
+          <mesh filename="package://dx_description/meshes/hand_bases/Config_1_Hand_Base.dae" />
+        </geometry>
+        <material name="">
+          <color rgba="0.898039215686275 0.917647058823529 0.929411764705882 1" />
+        </material>
+      </visual>
+      <collision>
+        <origin xyz="0 0 0" rpy="0 0 0" />
+        <geometry>
+          <mesh filename="package://dx_description/meshes/hand_bases/collision/Config_1_Hand_Base.stl" />
+        </geometry>
+      </collision>
+    </link>
+    <gazebo reference="${prefix}hand_base">
+      <selfCollide>true</selfCollide>
+    </gazebo>
+    <!-- Create a virtual end effector link that will be useful for arm IK -->
+    <link name="${prefix}end_effector"/>
+    <joint name="${prefix}ee_fixed_joint" type="fixed">
+      <parent link="${prefix}hand_base"/>
+      <child link="${prefix}end_effector"/>
+      <origin rpy="0.0 0.0 0.0" xyz="0.0 0.0 0.25"/>
+    </joint>
     <xacro:include filename="$(find dx_description)/xacros/dx_e3r3_finger.xacro" />
-    <xacro:macro_e3r3_finger prefix="${prefix}" finger_id="F0" parent="world">
-      <origin xyz="0 0.05 0.017" rpy="0 0 0"/>
+    <xacro:macro_e3r3_finger prefix="${prefix}" finger_id="F0" parent="${prefix}hand_base">
+      <origin xyz="0 0.05 0.017" rpy="-1.5707 0 0"/>
     </xacro:macro_e3r3_finger>
+    <xacro:include filename="$(find dx_description)/xacros/finger_blank.xacro" />
+    <xacro:macro_finger_blank prefix="${prefix}" finger_id="F1" parent="${prefix}hand_base">
+      <origin xyz="0.0384 -0.0287 0.017" rpy="-1.5707 0 -2.8159"/>
+    </xacro:macro_finger_blank>
+    <xacro:macro_finger_blank prefix="${prefix}" finger_id="F2" parent="${prefix}hand_base">
+      <origin xyz="-0.0384 -0.02870 0.017" rpy="-1.5707 0 2.8159"/>
+    </xacro:macro_finger_blank>
   </xacro:macro>
 </robot>

File: dx_description/xacros/finger_blank.xacro (robot description, xacro)
@@ -24,19 +24,36 @@
  software, even if advised of the possibility of such damage.
 -->
-<robot name="dexee_config_1_hand" xmlns:xacro="http://www.ros.org/wiki/xacro">
-  <xacro:include filename="$(find dx_description)/robot/0x02000106.xacro" />
-  <xacro:arg name="prefix" default="" />
-  <xacro:arg name="distal_type" default="sparkle" />  <!-- "sparkle" or "magtac" -->
-  <link name="world" />
-  <joint name="$(arg prefix)world_joint" type="fixed">
-    <parent link="world" />
-    <child link="$(arg prefix)hand_base" />
-  </joint>
-  <xacro:dexee_config_1_hand prefix="$(arg prefix)" distal_type="$(arg distal_type)" />
-  <gazebo>
-    <plugin name="gazebo_ros_control" filename="libgazebo_ros_control.so">
-        <!-- <robotNamespace>/</robotNamespace>
-        <legacyModeNS>false</legacyModeNS> -->
-    </plugin>
-  </gazebo>
+<robot xmlns:xacro="http://ros.org/wiki/xacro">
+  <xacro:macro name="macro_finger_blank" params="prefix:=^ finger_id parent *origin">
+    <joint name="${prefix}world_joint_${finger_id}" type="fixed">
+      <xacro:insert_block name="origin"/>
+      <parent link="${parent}" />
+      <child link="${prefix}${finger_id}_base" />
+    </joint>
+    <link name="${prefix}${finger_id}_base">
+      <inertial>
+        <origin rpy="1.5707 0 0" xyz="0.00008 -0.092 -0.00062"/>
+        <mass value="0.04087"/>
+        <inertia ixx="0.0004534284" ixy="-4.3115e-07" ixz="-3.57299999e-08" iyy="0.0000246748" iyz="0.0000321231" izz="0.0004555261"/>
+      </inertial>
+      <visual>
+        <origin xyz="0 0 0" rpy="1.5707 0 0" />
+        <geometry>
+          <mesh filename="package://dx_description/meshes/extras/Finger_blank.dae" />
+        </geometry>
+        <material name="">
+          <color rgba="0.75294 0.75294 0.75294 1" />
+        </material>
+      </visual>
+      <collision>
+        <origin xyz="0 0 0" rpy="1.5707 0 0" />
+        <geometry>
+          <mesh filename="package://dx_description/meshes/extras/collision/Finger_blank.stl" />
+        </geometry>
+      </collision>
+    </link>
+    <gazebo reference="${prefix}${finger_id}_base">
+      <selfCollide>true</selfCollide>
+    </gazebo>
+  </xacro:macro>
 </robot>
