Commit message: fix filepath typo

File: dx_description/xacros/distals/magtac.xacro (robot description, xacro)
@@ -35,5 +35,5 @@
         <origin xyz="0 0 0" rpy="0 0 0" />
         <geometry>
-            <mesh filename="package://dx_description/meshes/distal/magtac.dae" />
+            <mesh filename="package://dx_description/meshes/distals/magtac.dae" />
         </geometry>
         <material name="">

Commit message: re-orient distacs

File: dx_description/xacros/distals/magtac.xacro (robot description, xacro)
@@ -33,5 +33,5 @@
       </inertial>
       <visual>
-        <origin xyz="0 0 0" rpy="0 0 0" />
+        <origin xyz="0 0 0" rpy="-1.57079633 0 0" />
         <geometry>
             <mesh filename="package://dx_description/meshes/distals/magtac.dae" />
@@ -42,5 +42,5 @@
       </visual>
       <collision>
-        <origin xyz="0 0 0" rpy="0 0 0" />
+        <origin xyz="0 0 0" rpy="-1.57079633 0 0" />
         <geometry>
           <mesh filename="package://dx_description/meshes/distals/collision/magtac.stl" />
